File: public/kiCad/electrical/LogicGates/_autosave-LogicGates.kicad_sch (KiCad schematic)
At the start: 9 parts, among them Q1 NPN

Commit message: Logic Gate Update
Parts:
- removed C1, C2: 100nf, symbol Device:C
- removed R4: 390, symbol Device:R
- removed V2: VSIN, symbol Simulation_SPICE:VSIN
- added D1: D, symbol Simulation_SPICE:D
- added Q2: NPN, symbol Simulation_SPICE:NPN
- R1: value 1M -> 2k
- R2: value .1M -> 2k
- R3: value 10k -> 2k
- V1: value 9 -> 3.3
Connections:
- net 0: now also Q1.3 (E); no longer R2.2
- net at R1.1, R3.1, V1.1: now also R2.1
- net at Q1.1 (C): now also Q2.3 (E); no longer R3.2
- new net: D1.1 (K), Q2.1 (C)
- new net: D1.2 (A), R2.2
- new net: Q2.2 (B), R1.2
- new net: Q1.2 (B), R3.2
Other:
- title: (none) -> Logic Gates
